Commit message: added some boilerplate code for forklift joint controller into xacro, launch, and config yaml files

File: src/forklift_robot/urdf/ros2_control.xacro (robot description, xacro)
@@ -5,4 +5,5 @@
             <plugin>gazebo_ros2_control/GazeboSystem</plugin>
         </hardware>
+        <!-- Wheels -->
         <joint name="right_front_wheel_joint">
             <command_interface name="velocity">
@@ -17,4 +18,13 @@
                 <param name="min"> -10 </param>
                 <param name="max"> 10 </param>
+            </command_interface>
+            <state_interface name="velocity"/>
+            <state_interface name="position"/>
+        </joint>
+        <!-- Fork Joint -->
+        <joint name="fork_base_joint">
+            <command_interface name="position">
+              <param name="min">-1</param>
+              <param name="max">1</param>
             </command_interface>
             <state_interface name="velocity"/>

Commit message: fork_joint_controller now works and does not slide down.

File: src/forklift_robot/urdf/ros2_control.xacro (robot description, xacro)
@@ -29,5 +29,7 @@
             </command_interface>
             <command_interface name="velocity"/>
-            <command_interface name="position"/>
+            <command_interface name="position">
+                <!-- <limit effort="1000.0" lower="0" upper="0.38" velocity="10"/> -->
+            </command_interface>
             <!-- <state_interface name="velocity"/>
             <state_interface name="position"/> -->
