Commit message: Lidar plugin now works.

File: src/forklift_robot/urdf/gazebo_colors.xacro (robot description, xacro)
@@ -34,3 +34,6 @@
         <material>Gazebo/Red</material>
     </gazebo>
+    <gazebo reference="laser_frame_link">
+        <material>Gazebo/White</material>
+    </gazebo>
 </robot>

File: src/forklift_robot/urdf/lidar.xacro (robot description, xacro)
@@ -4,5 +4,5 @@
     <link name="laser_frame_link">
         <visual>
-            <origin xyz="0 0 ${laser_frame_length / 2}" rpy="0 0 0"/>
+            <origin xyz="0 0 0" rpy="0 0 0"/>
             <geometry>
                 <cylinder radius="${laser_frame_radius}" length="${laser_frame_length}"/>
@@ -13,5 +13,5 @@
         </visual>
         <collision>
-            <origin xyz="0 0 ${laser_frame_length / 2}" rpy="0 0 0"/>
+            <origin xyz="0 0 0" rpy="0 0 0"/>
             <geometry>
                 <cylinder radius="${laser_frame_radius}" length="laser_frame_length"/>
@@ -19,5 +19,5 @@
         </collision>
         <xacro:inertial_cylinder mass="${laser_frame_mass}" length="${laser_frame_length}" radius="${laser_frame_radius}">
-            <origin xyz="0 0 ${laser_frame_length / 2}" rpy="0 0 0"/>
+            <origin xyz="0 0 0" rpy="0 0 0"/>
         </xacro:inertial_cylinder>
     </link>
@@ -25,6 +25,34 @@
         <parent link="chassis_bottom_link"/>
         <child link="laser_frame_link"/>
-        <origin xyz=" 0 0 ${chassis_bottom_height + chassis_top_height}" rpy="0 0 0" />
+        <origin xyz=" 0 0 ${chassis_bottom_height + chassis_top_height + (laser_frame_length / 2)}" rpy="0 0 0" />
         <axis xyz="1 1 1"/>
     </joint>
+    <!-- Gazebo Plugin for Lidar -->
+    <gazebo reference="laser_frame_link">
+        <sensor name="laser" type="ray">
+            <pose> 0 0 0 0 0 0 </pose>
+            <visualize>true</visualize>
+            <update_rate>10</update_rate>
+            <ray>
+                <scan>
+                    <horizontal>
+                        <samples>360</samples>
+                        <min_angle>-3.14</min_angle>
+                        <max_angle>3.14</max_angle>
+                    </horizontal>
+                </scan>
+                <range>
+                    <min>0.3</min>
+                    <max>12</max>
+                </range>
+            </ray>
+            <plugin name="laser_controller" filename="libgazebo_ros_ray_sensor.so">
+                <ros>
+                    <argument>~/out:=scan</argument>
+                </ros>
+                <output_type>sensor_msgs/LaserScan</output_type>
+                <frame_name>laser_frame_link</frame_name>
+            </plugin>
+        </sensor>
+    </gazebo>
 </robot>
