Commit message: URDF for camera sensor added.

File: src/forklift_robot/urdf/camera.xacro (robot description, xacro)
@@ -1,10 +1,10 @@
 <?xml version="1.0"?>
 <robot xmlns:xacro="http://www.ros.org/wiki/xacro" >
-    <!-- Add link and a joint for the Lidar -->
-    <link name="laser_frame_link">
+    <!-- Add link and a joint for the CamerCamera -->
+    <link name="camera_link">
         <visual>
-            <origin xyz="0 0 0" rpy="0 0 0"/>
+            <origin xyz="${camera_size_x / 2} ${camera_size_y / 2} ${camera_size_z / 2}" rpy="0 0 0"/>
             <geometry>
-                <cylinder radius="${laser_frame_radius}" length="${laser_frame_length}"/>
+                <box size="${camera_size_x} ${camera_size_y} ${camera_size_z}"/>
             </geometry>
             <material name="white">
@@ -12,22 +12,13 @@
             </material>
         </visual>
-        <collision>
-            <origin xyz="0 0 0" rpy="0 0 0"/>
-            <geometry>
-                <cylinder radius="${laser_frame_radius}" length="laser_frame_length"/>
-            </geometry>
-        </collision>
-        <xacro:inertial_cylinder mass="${laser_frame_mass}" length="${laser_frame_length}" radius="${laser_frame_radius}">
-            <origin xyz="0 0 0" rpy="0 0 0"/>
-        </xacro:inertial_cylinder>
     </link>
-    <joint name="laser_frame_joint" type="fixed">
-        <parent link="chassis_bottom_link"/>
-        <child link="laser_frame_link"/>
-        <origin xyz=" 0 0 ${chassis_bottom_height + chassis_top_height + (laser_frame_length / 2)}" rpy="0 0 0" />
+    <joint name="camera_joint" type="fixed">
+        <parent link="fork_base_link"/>
+        <child link="camera_link"/>
+        <origin xyz="${fork_base_length / 2} ${fork_base_length / 2} ${fork_base_length / 2}" rpy="0 0 0"/>
     </joint>
-    <!-- Gazebo Plugin for Lidar -->
-    <gazebo reference="laser_frame_link">
-        <sensor name="laser" type="ray">
+    <!-- Gazebo Plugin for Camera -->
+    <gazebo reference="camera_link">
+        <!-- <sensor name="laser" type="ray">
             <pose> 0 0 0 0 0 0 </pose>
             <visualize>true</visualize>
@@ -53,5 +44,5 @@
                 <frame_name>laser_frame_link</frame_name>
             </plugin>
-        </sensor>
+        </sensor> -->
     </gazebo>
 </robot>

File: src/forklift_robot/urdf/forklift.urdf.xacro (robot description, xacro)
@@ -32,7 +32,11 @@
     <xacro:property name="laser_frame_length" value="0.04" />
     <xacro:property name="laser_frame_mass" value="0.01" />
+    <xacro:property name="camera_size_x" value="0.010" />
+    <xacro:property name="camera_size_y" value="0.03" />
+    <xacro:property name="camera_size_z" value="0.03" />
     <xacro:include filename="inertial_macros.xacro"/>
     <xacro:include filename="gazebo_colors.xacro"/>
     <xacro:include filename="lidar.xacro"/>
+    <xacro:include filename="camera.xacro"/>
     <!-- <xacro:include filename="gazebo.xacro"/> -->
     <!-- This first link called "world" is empty -->

File: src/forklift_robot/urdf/gazebo_colors.xacro (robot description, xacro)
@@ -37,3 +37,6 @@
         <material>Gazebo/White</material>
     </gazebo>
+    <gazebo reference="camera_link">
+        <material>Gazebo/White</material>
+    </gazebo>
 </robot>

Commit message: Camera plugin now works.

File: src/forklift_robot/urdf/camera.xacro (robot description, xacro)
@@ -1,5 +1,5 @@
 <?xml version="1.0"?>
 <robot xmlns:xacro="http://www.ros.org/wiki/xacro" >
-    <!-- Add link and a joint for the CamerCamera -->
+    <!-- Add link and a joint for the Camera -->
     <link name="camera_link">
         <visual>
@@ -16,33 +16,35 @@
         <parent link="fork_base_link"/>
         <child link="camera_link"/>
-        <origin xyz="${fork_base_length / 2} ${fork_base_length / 2} ${fork_base_length / 2}" rpy="0 0 0"/>
+        <origin xyz="${fork_base_length / 2} ${fork_base_length / 2} ${fork_base_length / 2}" rpy="0 0 ${pi / 2}"/> <!-- TODO: when the front of the robot faces x-axis(instead of current y-axis) change to rpy="0 0 0"-->
+    </joint>
+    <!-- Convert ros coordinate system to generally used image coordinate system -->
+    <link name="camera_link_optical"></link>
+    <joint name="camera_optical_joint" type="fixed">
+        <parent link="camera_link"/>
+        <child link="camera_link_optical"/>
+        <origin xyz="0 0 0" rpy="${-pi / 2} 0 ${-pi / 2}"/>
     </joint>
     <!-- Gazebo Plugin for Camera -->
     <gazebo reference="camera_link">
-        <!-- <sensor name="laser" type="ray">
+        <sensor name="camera" type="camera">
             <pose> 0 0 0 0 0 0 </pose>
             <visualize>true</visualize>
             <update_rate>10</update_rate>
-            <ray>
-                <scan>
-                    <horizontal>
-                        <samples>360</samples>
-                        <min_angle>-3.14</min_angle>
-                        <max_angle>3.14</max_angle>
-                    </horizontal>
-                </scan>
-                <range>
-                    <min>0.3</min>
-                    <max>12</max>
-                </range>
-            </ray>
-            <plugin name="laser_controller" filename="libgazebo_ros_ray_sensor.so">
-                <ros>
-                    <argument>~/out:=scan</argument>
-                </ros>
-                <output_type>sensor_msgs/LaserScan</output_type>
-                <frame_name>laser_frame_link</frame_name>
+            <camera>
+                <horizontal_fov>1.089</horizontal_fov>
+                <image>
+                    <format>R8G8B8</format>
+                    <width>${camera_image_width}</width> <!-- Width of the RGB image published by the camera sensor -->
+                    <height>${camera_image_height}</height> <!-- Height of the RGB image published by the camera sensor -->
+                </image>
+                <clip>
+                    <near>${camera_image_clip_near}</near> <!-- how close the camera can see -->
+                    <far>${camera_image_clip_far}</far> <!-- how far the camera can see -->
+                </clip>
+            </camera>
+            <plugin name="camera_controller" filename="libgazebo_ros_camera.so">
+                <frame_name>camera_link_optical</frame_name>
             </plugin>
-        </sensor> -->
+        </sensor>
     </gazebo>
 </robot>

File: src/forklift_robot/urdf/forklift.urdf.xacro (robot description, xacro)
@@ -35,4 +35,8 @@
     <xacro:property name="camera_size_y" value="0.03" />
     <xacro:property name="camera_size_z" value="0.03" />
+    <xacro:property name="camera_image_width" value="640" />  <!-- Width of the RGB image published by the camera sensor -->
+    <xacro:property name="camera_image_height" value="480" /> <!-- Height of the RGB image published by the camera sensor -->
+    <xacro:property name="camera_image_clip_near" value="0.05" /> <!-- how close the camera can see -->
+    <xacro:property name="camera_image_clip_far" value="8" /> <!-- how far the camera can see -->
     <xacro:include filename="inertial_macros.xacro"/>
     <xacro:include filename="gazebo_colors.xacro"/>
