Commit message: README.md added

File: src/forklift_robot/urdf/forklift.urdf.xacro (robot description, xacro)
@@ -1,33 +1,5 @@
 <?xml version="1.0"?>
 <robot xmlns:xacro="http://www.ros.org/wiki/xacro" name="forklift_bot">
-    <!-- <link name="world"></link>
-    <link name="base_link">
-        <inertial>
-            <origin xyz="0.0 0.0 0.0" rpy="0.0 0.0 0.0"/>
-            <mass value="0.0"/>
-            <inertia ixx="0.0" ixy="0.0" ixz="0.0" iyy="0.0" iyz="0.0" izz="0.0"/>
-        </inertial>
-        <visual name="temp">
-            <origin xyz="0.0 0.0 1.5" rpy="0.0 0.0 0.0"/>
-            <geometry>
-                <box size="2.0 4.0 3.0"/>
-            </geometry>
-            <material>
-                <color rgba="1.0 0.0 0.0 1.0"/>
-            </material>
-        </visual>
-        <collision>
-            <origin xyz="0.0 0.0 0.0" rpy="0.0 0.0 0.0"/>
-            <geometry>
-                <box size="0.0 0.0 0.0"/>
-            </geometry>
-        </collision>
-    </link>
-    <joint name="base_joint" type="fixed">
-        <origin xyz="1.5 1.0 0" rpy="0 0 0"/>
-        <parent link="world"/>
-        <child link="base_link"/>
-    </joint> -->
-    !-- This first link called "world" is empty -->
+    <!-- This first link called "world" is empty -->
     <link name="world"></link>
     <!-- A simple fixed joint from our empty world link, to our base. -->

Commit message: forklift_robot.xacro chassis and wheels added.

File: src/forklift_robot/urdf/forklift.urdf.xacro (robot description, xacro)
@@ -1,23 +1,33 @@
 <?xml version="1.0"?>
 <robot xmlns:xacro="http://www.ros.org/wiki/xacro" name="forklift_bot">
+    <xacro:property name="height_of_chassis_from_ground_plane" value="0.122" />
+    <xacro:property name="chassis_bottom_width" value="1.115" />
+    <xacro:property name="chassis_bottom_length" value="1.59" />
+    <xacro:property name="chassis_bottom_height" value="0.23" />
+    <xacro:property name="chassis_top_width" value="1.115" />
+    <xacro:property name="chassis_top_length" value="1.59" />
+    <xacro:property name="chassis_top_height" value="1.808" />
+    <xacro:include filename="inertial_macros.xacro"/>
+    <xacro:property name="back_wheel_radius" value="0.221" />
+    <xacro:property name="back_wheel_thickness" value="0.221" /> <!-- Made up number TODO: tune this parameter -->
+    <xacro:property name="back_wheel_mass" value="0.05" /> <!-- Made up number TODO: tune this parameter -->
+    <xacro:property name="back_wheel_length_offset" value="${(chassis_bottom_length / 2)  * (2/3)}" />
+    <xacro:property name="front_wheel_radius" value="0.30" />
+    <xacro:property name="front_wheel_thickness" value="0.23" /> <!-- Made up number TODO: tune this parameter -->
+    <xacro:property name="front_wheel_mass" value="0.05" /> <!-- Made up number TODO: tune this parameter -->
+    <xacro:property name="front_wheel_length_offset" value="${(chassis_bottom_length / 2)}" />
     <!-- This first link called "world" is empty -->
     <link name="world"></link>
-    <!-- A simple fixed joint from our empty world link, to our base. -->
-    <!-- The base origin is offset from the world origin. -->
-    <joint name="base_joint" type="fixed">
-        <origin xyz="1.5 1.0 0" rpy="0 0 0"/>
+    <!-- bottom of the chassis -->
+    <joint name="chassis_bottom_joint" type="fixed">
+        <origin xyz="1.5 1.0 ${height_of_chassis_from_ground_plane}" rpy="0 0 0"/>
         <parent link="world"/>
-        <child link="base_link"/>
+        <child link="chassis_bottom_link"/>
     </joint>
-    <!-- base_link is a large rectangular plate. Some things to note: -->
-    <!-- - We set the visual origin Z to half the box height, so that the link origin sits at the bottom of the box -->
-    <!-- - We set the collision to be identical to the visual -->
-    <!-- - We specified the colour manually (but still need to enter a name) -->
-    <!-- - We specified all the inertial parameters manually -->
-    <link name="base_link">
+    <link name="chassis_bottom_link">
         <visual>
-            <origin xyz="0 0 0.05" rpy="0 0 0"/>
+            <origin xyz="0 0 ${chassis_bottom_height / 2}" rpy="0 0 0"/>
             <geometry>
-                <box size="2.5 1.5 0.1" />
+                <box size="${chassis_bottom_width} ${chassis_bottom_length} ${chassis_bottom_height}" />
             </geometry>
             <material name="green">
@@ -26,14 +36,142 @@
         </visual>
         <collision>
-            <origin xyz="0 0 0.05" rpy="0 0 0"/>
+            <origin xyz="0 0 ${chassis_bottom_height / 2}" rpy="0 0 0"/>
             <geometry>
-                <box size="2.5 1.5 0.1" />
+                <box size="${chassis_bottom_width} ${chassis_bottom_length} ${chassis_bottom_height}" />
             </geometry>
         </collision>
         <inertial>
-            <origin xyz="0 0 0.05" rpy="0 0 0"/>
+            <origin xyz="0 0 0" rpy="0 0 0"/>
             <mass value="12" />
             <inertia ixx="2.26" ixy="0.0" ixz="0.0" iyy="6.26" iyz="0.0" izz="8.5" />
         </inertial>
     </link>
+    <!-- top of the chassis -->
+    <link name="chassis_top_link">
+        <visual>
+            <origin xyz="0 0 ${chassis_top_height / 2}" rpy="0 0 0"/>
+            <geometry>
+                <box size="${chassis_top_width} ${chassis_top_length} ${chassis_top_height}" />
+            </geometry>
+            <material name="red">
+                <color rgba="1 0 0 1"/>
+            </material>
+        </visual>
+        <collision>
+            <origin xyz="0 0 ${chassis_top_height / 2}" rpy="0 0 0"/>
+            <geometry>
+                <box size="${chassis_top_width} ${chassis_top_length} ${chassis_top_height}" />
+            </geometry>
+        </collision>
+        <inertial>
+            <origin xyz="0 0 0" rpy="0 0 0"/>
+            <mass value="12" />
+            <inertia ixx="2.26" ixy="0.0" ixz="0.0" iyy="6.26" iyz="0.0" izz="8.5" />
+        </inertial>
+    </link>
+    <joint name="chassis_top_joint" type="fixed">
+        <origin xyz="0 0 ${chassis_bottom_height}" rpy="0 0 0"/>
+        <parent link="chassis_bottom_link"/>
+        <child link="chassis_top_link"/>
+    </joint>
+    <!-- right_back_wheel -->
+    <link name="right_back_wheel_link">
+        <visual>
+            <geometry>
+                <cylinder radius="${back_wheel_radius}" length="${back_wheel_thickness}"/>
+            </geometry>
+            <material name="blue">
+                <color rgba="0 0 1 1"/>
+            </material>
+        </visual>
+        <collision>
+            <geometry>
+                <cylinder radius="${back_wheel_radius}" length="${back_wheel_thickness}"/>
+            </geometry>
+        </collision>
+        <xacro:inertial_cylinder mass="${back_wheel_mass}" length="${back_wheel_thickness}" radius="${back_wheel_radius}">
+            <origin xyz="0 0 0" rpy="0 0 0"/>
+        </xacro:inertial_cylinder>
+    </link>
+    <joint name="right_back_wheel_joint" type="continuous">
+        <parent link="chassis_bottom_link"/>
+        <child link="right_back_wheel_link"/>
+        <origin xyz="${(chassis_bottom_width / 2) - (back_wheel_thickness / 2)} -${back_wheel_length_offset} 0" rpy="0 -${pi/2} 0" />
+        <axis xyz="0 0 1"/>
+    </joint>
+    <!-- left_back_wheel -->
+    <link name="left_back_wheel_link">
+        <visual>
+            <geometry>
+                <cylinder radius="${back_wheel_radius}" length="${back_wheel_thickness}"/>
+            </geometry>
+            <material name="blue">
+                <color rgba="0 0 1 1"/>
+            </material>
+        </visual>
+        <collision>
+            <geometry>
+                <cylinder radius="${back_wheel_radius}" length="${back_wheel_thickness}"/>
+            </geometry>
+        </collision>
+        <xacro:inertial_cylinder mass="${back_wheel_mass}" length="${back_wheel_thickness}" radius="${back_wheel_radius}">
+            <origin xyz="0 0 0" rpy="0 0 0"/>
+        </xacro:inertial_cylinder>
+    </link>
+    <joint name="left_back_wheel_joint" type="continuous">
+        <parent link="chassis_bottom_link"/>
+        <child link="left_back_wheel_link"/>
+        <origin xyz="${- (chassis_bottom_width / 2) + (back_wheel_thickness / 2)} -${back_wheel_length_offset} 0" rpy="0 -${pi/2} 0" />
+        <axis xyz="0 0 1"/>
+    </joint>
+    <!-- right_front_wheel -->
+    <link name="right_front_wheel_link">
+        <visual>
+            <geometry>
+                <cylinder radius="${front_wheel_radius}" length="${front_wheel_thickness}"/>
+            </geometry>
+            <material name="blue">
+                <color rgba="0 0 1 1"/>
+            </material>
+        </visual>
+        <collision>
+            <geometry>
+                <cylinder radius="${front_wheel_radius}" length="${front_wheel_thickness}"/>
+            </geometry>
+        </collision>
+        <xacro:inertial_cylinder mass="${front_wheel_mass}" length="${front_wheel_thickness}" radius="${front_wheel_radius}">
+            <origin xyz="0 0 0" rpy="0 0 0"/>
+        </xacro:inertial_cylinder>
+    </link>
+    <joint name="right_front_wheel_joint" type="continuous">
+        <parent link="chassis_bottom_link"/>
+        <child link="right_front_wheel_link"/>
+        <origin xyz="${(chassis_bottom_width / 2) - (front_wheel_thickness / 2)} ${front_wheel_length_offset} 0" rpy="0 -${pi/2} 0" />
+        <axis xyz="0 0 1"/>
+    </joint>
+    <!-- left_front_wheel -->
+    <link name="left_front_wheel_link">
+        <visual>
+            <geometry>
+                <cylinder radius="${front_wheel_radius}" length="${front_wheel_thickness}"/>
+            </geometry>
+            <material name="blue">
+                <color rgba="0 0 1 1"/>
+            </material>
+        </visual>
+        <collision>
+            <geometry>
+                <cylinder radius="${front_wheel_radius}" length="${front_wheel_thickness}"/>
+            </geometry>
+        </collision>
+        <xacro:inertial_cylinder mass="${front_wheel_mass}" length="${front_wheel_thickness}" radius="${front_wheel_radius}">
+            <origin xyz="0 0 0" rpy="0 0 0"/>
+        </xacro:inertial_cylinder>
+    </link>
+    <joint name="left_front_wheel_joint" type="continuous">
+        <parent link="chassis_bottom_link"/>
+        <child link="left_front_wheel_link"/>
+        <origin xyz="${ -(chassis_bottom_width / 2) + (front_wheel_thickness / 2)} ${front_wheel_length_offset} 0" rpy="0 -${pi/2} 0" />
+        <axis xyz="0 0 1"/>
+    </joint>
 </robot>

Commit message: forklift_robot.xacro lift_base and forks are added. forklift functionality is implemented. TODO: Inertial tags should be set.

File: src/forklift_robot/urdf/forklift.urdf.xacro (robot description, xacro)
@@ -17,4 +17,17 @@
     <xacro:property name="front_wheel_mass" value="0.05" /> <!-- Made up number TODO: tune this parameter -->
     <xacro:property name="front_wheel_length_offset" value="${(chassis_bottom_length / 2)}" />
+    <xacro:property name="lift_body_connector_length" value="0.15" />
+    <xacro:property name="lift_base_length" value="0.25" />
+    <xacro:property name="lift_base_height" value="3.2" />
+    <xacro:property name="lift_body_connector_length" value="0.15" />
+    <xacro:property name="lift_body_connector_height" value="0.505" />
+    <xacro:property name="fork_base_width" value="1.050" />
+    <xacro:property name="fork_base_length" value="0.035" />
+    <xacro:property name="fork_base_height" value="1.220" />
+    <xacro:property name="fork_base_height_offset" value="${height_of_chassis_from_ground_plane - 0.076}" />
+    <xacro:property name="fork_length" value="0.99" />
+    <xacro:property name="fork_width" value="0.1" />
+    <xacro:property name="fork_height" value="0.045" />
+    <xacro:property name="fork_separation" value="0.850" /> <!-- separation (distance) between right fork and left fork -->
     <!-- This first link called "world" is empty -->
     <link name="world"></link>
@@ -175,3 +188,135 @@
         <axis xyz="0 0 1"/>
     </joint>
+    <!-- lift_base -->
+    <link name="lift_base_link">
+        <visual>
+            <origin xyz="0 0 ${lift_base_height / 2}" rpy="0 0 0"/>
+            <geometry>
+                <box size="${chassis_bottom_width} ${lift_base_length} ${lift_base_height}"/>
+            </geometry>
+            <material name="red">
+                <color rgba="1 0 0 1"/>
+            </material>
+        </visual>
+        <collision>
+            <origin xyz="0 0 ${lift_base_height / 2}" rpy="0 0 0"/>
+            <geometry>
+                <box size="${chassis_bottom_width} ${lift_base_length} ${lift_base_height}"/>
+            </geometry>
+        </collision>
+        <xacro:inertial_box mass="${front_wheel_mass}" x="0" y="0" z="0" > <!-- TODO: set weight etc. -->
+            <origin xyz="0 0 0" rpy="0 0 0"/>
+        </xacro:inertial_box>
+    </link>
+    <joint name="lift_base_joint" type="fixed">
+        <parent link="chassis_bottom_link"/>
+        <child link="lift_base_link"/>
+        <origin xyz="0 ${(chassis_bottom_length / 2) + lift_body_connector_length + (lift_base_length / 2)} 0" rpy="0 0 0" />
+    </joint>
+    <!-- lift_body_connector -->
+    <link name="lift_body_connector_link">
+        <visual>
+            <origin xyz="0 0 ${(lift_body_connector_height / 2)}" rpy="0 0 0"/>
+            <geometry>
+                <box size="${chassis_bottom_width} ${lift_body_connector_length} ${lift_body_connector_height}"/>
+            </geometry>
+            <material name="blue">
+                <color rgba="0 0 1 1"/>
+            </material>
+        </visual>
+        <collision>
+            <origin xyz="0 0 ${(lift_body_connector_height / 2)}" rpy="0 0 0"/>
+            <geometry>
+                <box size="${chassis_bottom_width} ${lift_body_connector_length} ${lift_body_connector_height}"/>
+            </geometry>
+        </collision>
+        <xacro:inertial_box mass="${front_wheel_mass}" x="0" y="0" z="0" > <!-- TODO: set weight etc. -->
+            <origin xyz="0 0 0" rpy="0 0 0"/>
+        </xacro:inertial_box>
+    </link>
+    <joint name="lift_body_connector_joint" type="fixed">
+        <parent link="chassis_bottom_link"/>
+        <child link="lift_body_connector_link"/>
+        <origin xyz="0 ${(chassis_bottom_length / 2) + (lift_body_connector_length / 2)} 0" rpy="0 0 0" />
+    </joint>
+    <!-- fork_base -->
+    <link name="fork_base_link">
+        <visual>
+            <origin xyz="0 0 ${(fork_base_height / 2)}" rpy="0 0 0"/>
+            <geometry>
+                <box size="${fork_base_width} ${fork_base_length} ${fork_base_height}"/>
+            </geometry>
+            <material name="green">
+                <color rgba="0 1 0 1"/>
+            </material>
+        </visual>
+        <collision>
+            <origin xyz="0 0 ${(fork_base_height / 2)}" rpy="0 0 0"/>
+            <geometry>
+                <box size="${fork_base_width} ${fork_base_length} ${fork_base_height}"/>
+            </geometry>
+        </collision>
+        <xacro:inertial_box mass="${front_wheel_mass}" x="0" y="0" z="0" > <!-- TODO: set weight etc. -->
+            <origin xyz="0 0 0" rpy="0 0 0"/>
+        </xacro:inertial_box>
+    </link>
+    <joint name="fork_base_joint" type="prismatic">
+        <parent link="lift_base_link"/>
+        <child link="fork_base_link"/>
+        <axis xyz="0 0 1"/>
+        <limit lower=" -${height_of_chassis_from_ground_plane - 0.015}" upper="${lift_base_height + fork_base_height_offset}" velocity="0.5" effort="1000.0"/> <!-- TODO: set limits -->
+        <origin xyz="0 ${(lift_base_length / 2) + (fork_base_length / 2)} -${fork_base_height_offset}" rpy="0 0 0"/>
+    </joint>
+    <!-- right_fork -->
+    <link name="right_fork_link">
+        <visual>
+            <origin xyz="0 0 ${(fork_height / 2)}" rpy="0 0 0"/>
+            <geometry>
+                <box size="${fork_width} ${fork_length} ${fork_height}"/>
+            </geometry>
+            <material name="red">
+                <color rgba="1 0 0 1"/>
+            </material>
+        </visual>
+        <collision>
+            <origin xyz="0 0 ${(fork_base_height / 2)}" rpy="0 0 0"/>
+            <geometry>
+                <box size="${fork_width} ${fork_length} ${fork_height}"/>
+            </geometry>
+        </collision>
+        <xacro:inertial_box mass="${front_wheel_mass}" x="0" y="0" z="0" > <!-- TODO: set weight etc. -->
+            <origin xyz="0 0 0" rpy="0 0 0"/>
+        </xacro:inertial_box>
+    </link>
+    <joint name="right_fork_joint" type="fixed">
+        <parent link="fork_base_link"/>
+        <child link="right_fork_link"/>
+        <origin xyz="${(fork_separation / 2) + (fork_width / 2)} ${(fork_base_length / 2) + (fork_length / 2)} 0" rpy="0 0 0"/>
+    </joint>
+    <!-- left_fork -->
+    <link name="left_fork_link">
+        <visual>
+            <origin xyz="0 0 ${(fork_height / 2)}" rpy="0 0 0"/>
+            <geometry>
+                <box size="${fork_width} ${fork_length} ${fork_height}"/>
+            </geometry>
+            <material name="red">
+                <color rgba="1 0 0 1"/>
+            </material>
+        </visual>
+        <collision>
+            <origin xyz="0 0 ${(fork_base_height / 2)}" rpy="0 0 0"/>
+            <geometry>
+                <box size="${fork_width} ${fork_length} ${fork_height}"/>
+            </geometry>
+        </collision>
+        <xacro:inertial_box mass="${front_wheel_mass}" x="0" y="0" z="0" > <!-- TODO: set weight etc. -->
+            <origin xyz="0 0 0" rpy="0 0 0"/>
+        </xacro:inertial_box>
+    </link>
+    <joint name="left_fork_joint" type="fixed">
+        <parent link="fork_base_link"/>
+        <child link="left_fork_link"/>
+        <origin xyz=" -${(fork_separation / 2) + (fork_width / 2)} ${(fork_base_length / 2) + (fork_length / 2)} 0" rpy="0 0 0"/>
+    </joint>
 </robot>

Commit message: gazebo_ros_joint_state_publisher and gazebo_ros_joint_pose_trajectory plugins added. Colors for gazebo are added. world frame is removed from forklift urdf.

File: src/forklift_robot/urdf/forklift.urdf.xacro (robot description, xacro)
@@ -1,4 +1,6 @@
 <?xml version="1.0"?>
 <robot xmlns:xacro="http://www.ros.org/wiki/xacro" name="forklift_bot">
+    <xacro:include filename="inertial_macros.xacro"/>
+    <xacro:include filename="gazebo.xacro"/>
     <xacro:property name="height_of_chassis_from_ground_plane" value="0.122" />
     <xacro:property name="chassis_bottom_width" value="1.115" />
@@ -8,5 +10,4 @@
     <xacro:property name="chassis_top_length" value="1.59" />
     <xacro:property name="chassis_top_height" value="1.808" />
-    <xacro:include filename="inertial_macros.xacro"/>
     <xacro:property name="back_wheel_radius" value="0.221" />
     <xacro:property name="back_wheel_thickness" value="0.221" /> <!-- Made up number TODO: tune this parameter -->
@@ -31,11 +32,11 @@
     <xacro:property name="fork_separation" value="0.850" /> <!-- separation (distance) between right fork and left fork -->
     <!-- This first link called "world" is empty -->
-    <link name="world"></link>
+    <!-- <link name="world"></link> -->
     <!-- bottom of the chassis -->
-    <joint name="chassis_bottom_joint" type="fixed">
+    <!-- <joint name="chassis_bottom_joint" type="fixed">
         <origin xyz="1.5 1.0 ${height_of_chassis_from_ground_plane}" rpy="0 0 0"/>
         <parent link="world"/>
         <child link="chassis_bottom_link"/>
-    </joint>
+    </joint> -->
     <link name="chassis_bottom_link">
         <visual>

Commit message: forklift model differential drive change.

File: src/forklift_robot/urdf/forklift.urdf.xacro (robot description, xacro)
@@ -90,5 +90,5 @@
     </joint>
     <!-- right_back_wheel -->
-    <link name="right_back_wheel_link">
+    <!-- <link name="right_back_wheel_link">
         <visual>
             <geometry>
@@ -113,7 +113,31 @@
         <origin xyz="${(chassis_bottom_width / 2) - (back_wheel_thickness / 2)} -${back_wheel_length_offset} 0" rpy="0 -${pi/2} 0" />
         <axis xyz="0 0 1"/>
+    </joint> -->
+    <link name="back_wheel_link">
+        <visual>
+            <geometry>
+                <sphere radius="${back_wheel_radius}"/>
+            </geometry>
+            <material name="blue">
+                <color rgba="0 0 1 1"/>
+            </material>
+        </visual>
+        <collision>
+            <geometry>
+                <sphere radius="${back_wheel_radius}"/>
+            </geometry>
+        </collision>
+        <xacro:inertial_cylinder mass="${back_wheel_mass}" length="${back_wheel_thickness}" radius="${back_wheel_radius}">
+            <origin xyz="0 0 0" rpy="0 0 0"/>
+        </xacro:inertial_cylinder>
+    </link>
+    <joint name="back_wheel_joint" type="continuous">
+        <parent link="chassis_bottom_link"/>
+        <child link="back_wheel_link"/>
+        <origin xyz=" 0 -${back_wheel_length_offset} 0" rpy="0 -${pi/2} 0" />
+        <axis xyz="1 1 1"/>
     </joint>
     <!-- left_back_wheel -->
-    <link name="left_back_wheel_link">
+    <!-- <link name="left_back_wheel_link">
         <visual>
             <geometry>
@@ -138,5 +162,5 @@
         <origin xyz="${- (chassis_bottom_width / 2) + (back_wheel_thickness / 2)} -${back_wheel_length_offset} 0" rpy="0 -${pi/2} 0" />
         <axis xyz="0 0 1"/>
-    </joint>
+    </joint> -->
     <!-- right_front_wheel -->
     <link name="right_front_wheel_link">

File: src/forklift_robot/urdf/gazebo.xacro (robot description, xacro)
@@ -115,11 +115,13 @@
     <xacro:property name="back_wheel_thickness" value="0.221" /> <!-- Made up number TODO: tune this parameter -->
     <xacro:property name="back_wheel_radius" value="0.221" />
+    <xacro:property name="front_wheel_radius" value="0.30" />
+    <xacro:property name="front_wheel_thickness" value="0.23" /> <!-- Made up number TODO: tune this parameter -->
     <gazebo>
         <plugin name="diff_drive" filename="libgazebo_ros_diff_drive.so">
             <!-- Wheel Information -->
-            <left_joint>right_back_wheel_joint</left_joint>
-            <right_joint>left_back_wheel_joint</right_joint>
-            <wheel_separation>${chassis_bottom_width - back_wheel_thickness}</wheel_separation>
-            <wheel_diameter>${back_wheel_radius * 2}</wheel_diameter>
+            <left_joint>right_front_wheel_joint</left_joint>
+            <right_joint>left_front_wheel_joint</right_joint>
+            <wheel_separation>${chassis_bottom_width - front_wheel_thickness}</wheel_separation>
+            <wheel_diameter>${front_wheel_radius * 2}</wheel_diameter>
             <!-- Limits -->
             <max_wheel_torque>200</max_wheel_torque>
