Commit message: gazebo.xacro xacro property imports fixed

File: src/forklift_robot/urdf/forklift.urdf.xacro (robot description, xacro)
@@ -1,6 +1,4 @@
 <?xml version="1.0"?>
 <robot xmlns:xacro="http://www.ros.org/wiki/xacro" name="forklift_bot">
-    <xacro:include filename="inertial_macros.xacro"/>
-    <xacro:include filename="gazebo.xacro"/>
     <xacro:property name="height_of_chassis_from_ground_plane" value="0.122" />
     <xacro:property name="chassis_bottom_width" value="1.115" />
@@ -31,4 +29,6 @@
     <xacro:property name="fork_height" value="0.045" />
     <xacro:property name="fork_separation" value="0.850" /> <!-- separation (distance) between right fork and left fork -->
+    <xacro:include filename="inertial_macros.xacro"/>
+    <xacro:include filename="gazebo.xacro"/>
     <!-- This first link called "world" is empty -->
     <!-- <link name="world"></link> -->

File: src/forklift_robot/urdf/gazebo.xacro (robot description, xacro)
@@ -112,9 +112,9 @@
     </gazebo> -->
     <!-- Control plugins from another video -->
-    <xacro:property name="chassis_bottom_width" value="1.115" />
-    <xacro:property name="back_wheel_thickness" value="0.221" /> <!-- Made up number TODO: tune this parameter -->
+    <!-- <xacro:property name="chassis_bottom_width" value="1.115" />
+    <xacro:property name="back_wheel_thickness" value="0.221" /> Made up number TODO: tune this parameter
     <xacro:property name="back_wheel_radius" value="0.221" />
     <xacro:property name="front_wheel_radius" value="0.30" />
-    <xacro:property name="front_wheel_thickness" value="0.23" /> <!-- Made up number TODO: tune this parameter -->
+    <xacro:property name="front_wheel_thickness" value="0.23" /> Made up number TODO: tune this parameter -->
     <gazebo>
         <plugin name="diff_drive" filename="libgazebo_ros_diff_drive.so">
@@ -122,5 +122,5 @@
             <left_joint>right_front_wheel_joint</left_joint>
             <right_joint>left_front_wheel_joint</right_joint>
-            <wheel_separation>${chassis_bottom_width - front_wheel_thickness}</wheel_separation>
+            <wheel_separation>${chassis_bottom_width - (2*front_wheel_thickness)}</wheel_separation>
             <wheel_diameter>${front_wheel_radius * 2}</wheel_diameter>
             <!-- Limits -->

Commit message: ros2_control tags added to forklift_robot urdf file. differential_drive control configs for ros2_control added.

File: src/forklift_robot/urdf/forklift.urdf.xacro (robot description, xacro)
@@ -347,4 +347,4 @@
     </joint>
     <!-- Setup ROS_CONTROL and transmission tags -->
-    <xacro:include filename="ros_control.xacro"/>
+    <xacro:include filename="ros2_control.xacro"/>
 </robot>

File: src/forklift_robot/urdf/ros2_control.xacro (robot description, xacro)
@@ -1,6 +1,33 @@
 <?xml version="1.0"?>
 <robot xmlns:xacro="http://www.ros.org/wiki/xacro" >
+    <ros2_control name="GazeboSystem" type="system">
+        <hardware>
+            <plugin>gazebo_ros2_control/GazeboSystem</plugin>
+        </hardware>
+        <joint name="right_front_wheel_joint">
+            <command_interface name="velocity">
+                <param name="min"> -10 </param>
+                <param name="max"> 10 </param>
+            </command_interface>
+            <state_interface name="velocity"/>
+            <state_interface name="positiion"/>
+        </joint>
+        <joint name="left_front_wheel_joint">
+            <command_interface name="velocity">
+                <param name="min"> -10 </param>
+                <param name="max"> 10 </param>
+            </command_interface>
+            <state_interface name="velocity"/>
+            <state_interface name="positiion"/>
+        </joint>
+    </ros2_control>
+    <gazebo>
+        <plugin name="gazebo_ros2_control" filename="libgazebo_ros2_control.so">
+            <parameters>$(find forklift_robot)/my_controllers.yaml</parameters>
+            <!-- <parameters>$(find forklift_robot)/config/my_controllers.yaml</parameters> -->
+        </plugin>
+    </gazebo>
     <!-- Add transmission tags for forklift URDF bot -->
-    <transmission name="transmission_right_front_wheel_joint">
+    <!-- <transmission name="transmission_right_front_wheel_joint">
         <type>transmission_interface/SimpleTransmission</type>
         <joint name="right_front_wheel_joint">
@@ -21,7 +48,7 @@
             <mechanicalReduction>1</mechanicalReduction>
         </actuator>
-    </transmission>
+    </transmission> -->
     <!-- Include Ros_Control for Gazebo Simulation plugin -->
-    <gazebo>
+    <!-- <gazebo>
         <plugin filename="libgazebo_ros2_control.so" name="gazebo_ros2_control">
             <robot_param>robot_description</robot_param>
@@ -29,10 +56,4 @@
             <parameters>$(find forklift_ros_control)/config/forklift_control.yaml</parameters>
         </plugin>
-    </gazebo>
-    <!-- <gazebo>
-        <plugin name="gazebo_ros_control" filename="libgazebo_ros_control.so">
-            <robotNamespace>/ForkliftBot</robotNamespace>
-            <robotSimType>gazebo_ros_control/DefaultRobotHWSim</robotSimType>
-        </plugin>
     </gazebo> -->
 </robot>

Commit message: bug fix: collision origin tag of left_fork_link and right_fork_link fixed.

File: src/forklift_robot/urdf/forklift.urdf.xacro (robot description, xacro)
@@ -306,5 +306,5 @@
         </visual>
         <collision>
-            <origin xyz="0 0 ${(fork_base_height / 2)}" rpy="0 0 0"/>
+            <origin xyz="0 0 ${(fork_height / 2)}" rpy="0 0 0"/>
             <geometry>
                 <box size="${fork_width} ${fork_length} ${fork_height}"/>
@@ -332,5 +332,5 @@
         </visual>
         <collision>
-            <origin xyz="0 0 ${(fork_base_height / 2)}" rpy="0 0 0"/>
+            <origin xyz="0 0 ${(fork_height / 2)}" rpy="0 0 0"/>
             <geometry>
                 <box size="${fork_width} ${fork_length} ${fork_height}"/>

File: src/forklift_robot/urdf/gazebo.xacro (robot description, xacro)
@@ -120,6 +120,6 @@
         <plugin name="diff_drive" filename="libgazebo_ros_diff_drive.so">
             <!-- Wheel Information -->
-            <left_joint>right_front_wheel_joint</left_joint>
-            <right_joint>left_front_wheel_joint</right_joint>
+            <left_joint>left_front_wheel_joint</left_joint>
+            <right_joint>right_front_wheel_joint</right_joint>
             <wheel_separation>${chassis_bottom_width - (2*front_wheel_thickness)}</wheel_separation>
             <wheel_diameter>${front_wheel_radius * 2}</wheel_diameter>

Commit message: URDF for Lidar sensor added.

File: src/forklift_robot/urdf/forklift.urdf.xacro (robot description, xacro)
@@ -29,6 +29,10 @@
     <xacro:property name="fork_height" value="0.045" />
     <xacro:property name="fork_separation" value="0.850" /> <!-- separation (distance) between right fork and left fork -->
+    <xacro:property name="laser_frame_radius" value="0.05" />
+    <xacro:property name="laser_frame_length" value="0.04" />
+    <xacro:property name="laser_frame_mass" value="0.01" />
     <xacro:include filename="inertial_macros.xacro"/>
     <xacro:include filename="gazebo_colors.xacro"/>
+    <xacro:include filename="lidar.xacro"/>
     <!-- <xacro:include filename="gazebo.xacro"/> -->
     <!-- This first link called "world" is empty -->

Commit message: @fix: forklift moving weidly issue fixed. To solve it back_wheel is changed.

File: src/forklift_robot/urdf/forklift.urdf.xacro (robot description, xacro)
@@ -146,10 +146,15 @@
         </xacro:inertial_cylinder>
     </link>
-    <joint name="back_wheel_joint" type="continuous">
+    <joint name="back_wheel_joint" type="fixed">
+        <parent link="chassis_bottom_link"/>
+        <child link="back_wheel_link"/>
+        <origin xyz=" 0 -${back_wheel_length_offset} 0" rpy="0 -${pi/2} 0" />
+    </joint>
+    <!-- <joint name="back_wheel_joint" type="continuous">
         <parent link="chassis_bottom_link"/>
         <child link="back_wheel_link"/>
         <origin xyz=" 0 -${back_wheel_length_offset} 0" rpy="0 -${pi/2} 0" />
         <axis xyz="1 1 1"/>
-    </joint>
+    </joint> -->
     <!-- left_back_wheel -->
     <!-- <link name="left_back_wheel_link">

File: src/forklift_robot/urdf/gazebo_colors.xacro (robot description, xacro)
@@ -40,3 +40,8 @@
         <material>Gazebo/White</material>
     </gazebo>
+    <gazebo reference="back_wheel_link">
+        <material>Gazebo/White</material>
+        <mu1 value="0.001"/> <!-- Reduce Friction to use it as a Caster Wheel -->
+        <mu2 value="0.001"/>
+    </gazebo>
 </robot>

Commit message: OpenAI GYM environment reset bug

File: src/forklift_robot/urdf/forklift.urdf.xacro (robot description, xacro)
@@ -8,6 +8,8 @@
     <xacro:property name="chassis_top_length" value="1.59" />
     <xacro:property name="chassis_top_height" value="1.808" />
-    <xacro:property name="back_wheel_radius" value="0.221" />
-    <xacro:property name="back_wheel_thickness" value="0.221" /> <!-- Made up number TODO: tune this parameter -->
+    <!-- <xacro:property name="back_wheel_radius" value="0.221" />
+    <xacro:property name="back_wheel_thickness" value="0.221" />  -->
+    <xacro:property name="back_wheel_radius" value="0.30" />
+    <xacro:property name="back_wheel_thickness" value="0.23" /> <!-- Made up number TODO: tune this parameter -->
     <xacro:property name="back_wheel_mass" value="0.05" /> <!-- Made up number TODO: tune this parameter -->
     <xacro:property name="back_wheel_length_offset" value="${(chassis_bottom_length / 2)  * (2/3)}" />
@@ -49,5 +51,5 @@
     <!-- bottom of the chassis -->
     <!-- <joint name="chassis_bottom_joint" type="fixed">
-        <origin xyz="1.5 1.0 ${height_of_chassis_from_ground_plane}" rpy="0 0 0"/>
+        <origin xyz="0 0 ${height_of_chassis_from_ground_plane}" rpy="0 0 0"/>
         <parent link="world"/>
         <child link="chassis_bottom_link"/>
@@ -94,5 +96,5 @@
         <inertial>
             <origin xyz="0 0 0" rpy="0 0 0"/>
-            <mass value="12" />
+            <mass value="12" />221
             <inertia ixx="2.26" ixy="0.0" ixz="0.0" iyy="6.26" iyz="0.0" izz="8.5" />
         </inertial>

Commit message: gui_controller for controlling forklift robot manually.

File: src/forklift_robot/urdf/forklift.urdf.xacro (robot description, xacro)
@@ -43,7 +43,7 @@
     <xacro:include filename="inertial_macros.xacro"/>
     <xacro:include filename="gazebo_colors.xacro"/>
-    <xacro:include filename="lidar.xacro"/>
+    <!-- <xacro:include filename="lidar.xacro"/> -->
     <!-- <xacro:include filename="camera.xacro"/> --> <!-- Uncomment this line, and comment the line below to switch between Depth Camera and a Regular Camera -->
-    <xacro:include filename="depth_camera.xacro"/>
+    <!-- <xacro:include filename="depth_camera.xacro"/> -->
     <!-- <xacro:include filename="gazebo.xacro"/> -->
     <!-- This first link called "world" is empty -->
@@ -250,4 +250,18 @@
                 <box size="${chassis_bottom_width} ${lift_base_length} ${lift_base_height}"/>
             </geometry>
+            <!-- Added by me (surface tag) to prevent fork falling down issue -->
+            <surface>
+                <friction>
+                    <ode>
+                        <mu>100000.0</mu> <!-- TODO: set mu values -->
+                        <mu2>100000.0</mu2>
+                    </ode>
+                </friction>
+                <contact>
+                    <ode>
+                        <min_depth>0.003</min_depth>
+                    </ode>
+                </contact>
+            </surface>
         </collision>
         <xacro:inertial_box mass="${front_wheel_mass}" x="0" y="0" z="0" > <!-- TODO: set weight etc. -->
@@ -302,4 +316,18 @@
                 <box size="${fork_base_width} ${fork_base_length} ${fork_base_height}"/>
             </geometry>
+            <!-- Added by me (surface tag) to prevent fork falling down issue -->
+            <surface>
+                <friction>
+                    <ode>
+                        <mu>100000.0</mu> <!-- TODO: set mu values-->
+                        <mu2>100000.0</mu2>
+                    </ode>
+                </friction>
+                <contact>
+                    <ode>
+                        <min_depth>0.003</min_depth>
+                    </ode>
+                </contact>
+            </surface>
         </collision>
         <xacro:inertial_box mass="${front_wheel_mass}" x="0" y="0" z="0" > <!-- TODO: set weight etc. -->

File: src/forklift_robot/urdf/ros2_control.xacro (robot description, xacro)
@@ -30,4 +30,5 @@
             <command_interface name="velocity"/>
             <command_interface name="position">
+                <!-- <limit effort="87" lower="-1.7628" upper="1.7628" velocity="2.1750"/>  -->
                 <!-- <limit effort="1000.0" lower="0" upper="0.38" velocity="10"/> -->
             </command_interface>

Commit message: ros_collision_detection plugin integration to forklift_robot, automate exporting GAZEBO_PLUGIN_PATH env variable.

File: src/forklift_robot/urdf/forklift.urdf.xacro (robot description, xacro)
@@ -65,5 +65,5 @@
             </material>
         </visual>
-        <collision>
+        <collision name="chassis_bottom_link_collision">
             <origin xyz="0 0 ${chassis_bottom_height / 2}" rpy="0 0 0"/>
             <geometry>
@@ -77,4 +77,16 @@
         </inertial>
     </link>
+    <gazebo reference="chassis_bottom_link">
+        <sensor name='my_contact' type='contact'>
+            <plugin name="my_plugin3" filename="libros_collision_detection.so"/>
+            <update_rate> 30.0 </update_rate>
+            <selfCollide>true</selfCollide>
+            <alwaysOn>true</alwaysOn>
+            <material>Gazebo/White</material>
+            <contact>
+                <collision>chassis_bottom_link_collision_collision</collision>
+            </contact>
+        </sensor>
+    </gazebo>
     <!-- top of the chassis -->
     <link name="chassis_top_link">

Commit message: ros_collision_detection_plugin forklift_env reset issue fixed

File: src/forklift_robot/urdf/forklift.urdf.xacro (robot description, xacro)
@@ -41,4 +41,5 @@
     <xacro:property name="camera_image_clip_near" value="0.05" /> <!-- how close the camera can see -->
     <xacro:property name="camera_image_clip_far" value="8" /> <!-- how far the camera can see -->
+    <xacro:property name="collision_detection_plugin_update_rate" value="30.0" /> <!-- how far the camera can see -->
     <xacro:include filename="inertial_macros.xacro"/>
     <xacro:include filename="gazebo_colors.xacro"/>
@@ -77,16 +78,4 @@
         </inertial>
     </link>
-    <gazebo reference="chassis_bottom_link">
-        <sensor name='my_contact' type='contact'>
-            <plugin name="my_plugin3" filename="libros_collision_detection.so"/>
-            <update_rate> 30.0 </update_rate>
-            <selfCollide>true</selfCollide>
-            <alwaysOn>true</alwaysOn>
-            <material>Gazebo/White</material>
-            <contact>
-                <collision>chassis_bottom_link_collision_collision</collision>
-            </contact>
-        </sensor>
-    </gazebo>
     <!-- top of the chassis -->
     <link name="chassis_top_link">
@@ -408,3 +397,5 @@
     <!-- Setup ROS_CONTROL and transmission tags -->
     <xacro:include filename="ros2_control.xacro"/>
+    <!-- Setup Collision Detection Plugin for the forklift robot -->
+    <xacro:include filename="ros_gazebo_collision_detection_plugin.xacro"/>
 </robot>

Commit message: diff_drive left and right turn issue fixed

File: src/forklift_robot/urdf/forklift.urdf.xacro (robot description, xacro)
@@ -74,5 +74,5 @@
         <inertial>
             <origin xyz="0 0 0" rpy="0 0 0"/>
-            <mass value="12" />
+            <mass value="120" />
             <inertia ixx="2.26" ixy="0.0" ixz="0.0" iyy="6.26" iyz="0.0" izz="8.5" />
         </inertial>
@@ -149,9 +149,19 @@
         </xacro:inertial_cylinder>
     </link>
-    <joint name="back_wheel_joint" type="fixed">
+    <!-- <joint name="back_wheel_joint" type="fixed">
         <parent link="chassis_bottom_link"/>
         <child link="back_wheel_link"/>
         <origin xyz=" 0 -${back_wheel_length_offset} 0" rpy="0 -${pi/2} 0" />
-    </joint>
+    </joint> -->
+    <joint name="back_wheel_joint" type="fixed">
+        <parent link="chassis_bottom_link"/>
+        <child link="back_wheel_link"/>
+        <origin xyz=" 0 -${back_wheel_length_offset} 0" />
+    </joint>
+    <gazebo reference="back_wheel_link">
+        <material>Gazebo/White</material>
+        <mu1 value="0.001"/>
+        <mu2 value="0.001"/>
+    </gazebo>
     <!-- <joint name="back_wheel_joint" type="continuous">
         <parent link="chassis_bottom_link"/>
