Commit message: inertia values for forklift changed

File: src/forklift_robot/urdf/forklift.urdf.xacro (robot description, xacro)
@@ -12,9 +12,9 @@
     <xacro:property name="back_wheel_radius" value="0.30" />
     <xacro:property name="back_wheel_thickness" value="0.23" /> <!-- Made up number TODO: tune this parameter -->
-    <xacro:property name="back_wheel_mass" value="0.05" /> <!-- Made up number TODO: tune this parameter -->
+    <xacro:property name="back_wheel_mass" value="0.01" /> <!-- Made up number TODO: tune this parameter -->
     <xacro:property name="back_wheel_length_offset" value="${(chassis_bottom_length / 2)  * (2/3)}" />
     <xacro:property name="front_wheel_radius" value="0.30" />
     <xacro:property name="front_wheel_thickness" value="0.23" /> <!-- Made up number TODO: tune this parameter -->
-    <xacro:property name="front_wheel_mass" value="0.05" /> <!-- Made up number TODO: tune this parameter -->
+    <xacro:property name="front_wheel_mass" value="0.005" /> <!-- Made up number TODO: tune this parameter -->
     <xacro:property name="front_wheel_length_offset" value="${(chassis_bottom_length / 2)}" />
     <xacro:property name="lift_body_connector_length" value="0.15" />
@@ -47,12 +47,11 @@
     <!-- <xacro:include filename="camera.xacro"/> --> <!-- Uncomment this line, and comment the line below to switch between Depth Camera and a Regular Camera -->
     <xacro:include filename="depth_camera.xacro"/>
-    <!-- <xacro:include filename="gazebo.xacro"/> -->
-    <!-- This first link called "world" is empty -->
-    <!-- <link name="world"></link> -->
-    <!-- bottom of the chassis -->
-    <!-- <joint name="chassis_bottom_joint" type="fixed">
-        <origin xyz="0 0 ${height_of_chassis_from_ground_plane}" rpy="0 0 0"/>
-        <parent link="world"/>
+    <!-- BASE LINK -->
+    <!-- <link name="base_link">
+    </link>
+    <joint name="chassis_joint" type="fixed">
+        <parent link="base_link"/>
         <child link="chassis_bottom_link"/>
+        <origin xyz="0 0 0"/>
     </joint> -->
     <link name="chassis_bottom_link">
@@ -72,9 +71,7 @@
             </geometry>
         </collision>
-        <inertial>
-            <origin xyz="0 0 0" rpy="0 0 0"/>
-            <mass value="120" />
-            <inertia ixx="2.26" ixy="0.0" ixz="0.0" iyy="6.26" iyz="0.0" izz="8.5" />
-        </inertial>
+        <xacro:inertial_box mass="1" x="${chassis_bottom_width}" y="${chassis_bottom_length}" z="${chassis_bottom_height}">
+            <origin xyz="0 0 ${chassis_bottom_height / 2}" rpy="0 0 0"/>
+        </xacro:inertial_box>
     </link>
     <!-- top of the chassis -->
@@ -95,9 +92,7 @@
             </geometry>
         </collision>
-        <inertial>
-            <origin xyz="0 0 0" rpy="0 0 0"/>
-            <mass value="12" />221
-            <inertia ixx="2.26" ixy="0.0" ixz="0.0" iyy="6.26" iyz="0.0" izz="8.5" />
-        </inertial>
+        <xacro:inertial_box mass="5" x="${chassis_top_width}" y="${chassis_top_length}" z="${chassis_top_height}">
+            <origin xyz="0 0 ${chassis_top_height / 2}" rpy="0 0 0"/>
+        </xacro:inertial_box>
     </link>
     <joint name="chassis_top_joint" type="fixed">
@@ -145,7 +140,7 @@
             </geometry>
         </collision>
-        <xacro:inertial_cylinder mass="${back_wheel_mass}" length="${back_wheel_thickness}" radius="${back_wheel_radius}">
+        <xacro:inertial_sphere mass="${back_wheel_mass}" radius="${back_wheel_radius}">
             <origin xyz="0 0 0" rpy="0 0 0"/>
-        </xacro:inertial_cylinder>
+        </xacro:inertial_sphere>
     </link>
     <!-- <joint name="back_wheel_joint" type="fixed">
@@ -159,4 +154,5 @@
         <origin xyz=" 0 -${back_wheel_length_offset} 0" />
     </joint>
+    <!-- Wheel Frictions -->
     <gazebo reference="back_wheel_link">
         <material>Gazebo/White</material>
@@ -164,10 +160,14 @@
         <mu2 value="0.001"/>
     </gazebo>
-    <!-- <joint name="back_wheel_joint" type="continuous">
-        <parent link="chassis_bottom_link"/>
-        <child link="back_wheel_link"/>
-        <origin xyz=" 0 -${back_wheel_length_offset} 0" rpy="0 -${pi/2} 0" />
-        <axis xyz="1 1 1"/>
-    </joint> -->
+    <gazebo reference="right_front_wheel_link">
+        <material>Gazebo/White</material>
+        <mu1 value="1.0"/>
+        <mu2 value="0.25"/>
+    </gazebo>
+    <gazebo reference="left_front_wheel_link">
+        <material>Gazebo/White</material>
+        <mu1 value="1.0"/>
+        <mu2 value="0.25"/>
+    </gazebo>
     <!-- left_back_wheel -->
     <!-- <link name="left_back_wheel_link">
@@ -217,6 +217,8 @@
         <parent link="chassis_bottom_link"/>
         <child link="right_front_wheel_link"/>
-        <origin xyz="${(chassis_bottom_width / 2) - (front_wheel_thickness / 2)} ${front_wheel_length_offset} 0" rpy="0 -${pi/2} 0" />
-        <axis xyz="0 0 1"/>
+        <!-- <origin xyz="${(chassis_bottom_width / 2) - (front_wheel_thickness / 2)} ${front_wheel_length_offset} 0" rpy="0 ${pi/2} 0" /> -->
+        <origin xyz="${(chassis_bottom_width / 2)} ${front_wheel_length_offset} 0" rpy="0 ${pi/2} 0" />
+        <axis xyz="0 0 -1"/>
+        <dynamics damping="0.2"/>
     </joint>
     <!-- left_front_wheel -->
@@ -242,6 +244,8 @@
         <parent link="chassis_bottom_link"/>
         <child link="left_front_wheel_link"/>
-        <origin xyz="${ -(chassis_bottom_width / 2) + (front_wheel_thickness / 2)} ${front_wheel_length_offset} 0" rpy="0 -${pi/2} 0" />
+        <!-- <origin xyz="${ -(chassis_bottom_width / 2) + (front_wheel_thickness / 2)} ${front_wheel_length_offset} 0" rpy="0 -${pi/2} 0" /> -->
+        <origin xyz="${ -(chassis_bottom_width / 2)} ${front_wheel_length_offset} 0" rpy="0 -${pi/2} 0" />
         <axis xyz="0 0 1"/>
+        <dynamics damping="0.2"/>
     </joint>
     <!-- lift_base -->
@@ -262,8 +266,8 @@
             </geometry>
             <!-- Added by me (surface tag) to prevent fork falling down issue -->
-            <surface>
+            <!-- <surface>
                 <friction>
                     <ode>
-                        <mu>100000.0</mu> <!-- TODO: set mu values -->
+                        <mu>100000.0</mu>
                         <mu2>100000.0</mu2>
                     </ode>
@@ -274,8 +278,8 @@
                     </ode>
                 </contact>
-            </surface>
-        </collision>
-        <xacro:inertial_box mass="${front_wheel_mass}" x="0" y="0" z="0" > <!-- TODO: set weight etc. -->
-            <origin xyz="0 0 0" rpy="0 0 0"/>
+            </surface> -->
+        </collision>
+        <xacro:inertial_box mass="${0.001}" x="${chassis_bottom_width}" y="${lift_base_length}" z="${lift_base_height}" >
+            <origin xyz="0 0 ${lift_base_height / 2}" rpy="0 0 0"/>
         </xacro:inertial_box>
     </link>
@@ -302,6 +306,6 @@
             </geometry>
         </collision>
-        <xacro:inertial_box mass="${front_wheel_mass}" x="0" y="0" z="0" > <!-- TODO: set weight etc. -->
-            <origin xyz="0 0 0" rpy="0 0 0"/>
+        <xacro:inertial_box mass="${0.001}" x="${chassis_bottom_width}" y="${lift_body_connector_length}" z="${lift_body_connector_height}" >
+            <origin xyz="0 0 ${(lift_body_connector_height / 2)}" rpy="0 0 0"/>
         </xacro:inertial_box>
     </link>
@@ -328,8 +332,8 @@
             </geometry>
             <!-- Added by me (surface tag) to prevent fork falling down issue -->
-            <surface>
+            <!-- <surface>
                 <friction>
                     <ode>
-                        <mu>100000.0</mu> <!-- TODO: set mu values-->
+                        <mu>100000.0</mu>
                         <mu2>100000.0</mu2>
                     </ode>
@@ -340,8 +344,8 @@
                     </ode>
                 </contact>
-            </surface>
-        </collision>
-        <xacro:inertial_box mass="${front_wheel_mass}" x="0" y="0" z="0" > <!-- TODO: set weight etc. -->
-            <origin xyz="0 0 0" rpy="0 0 0"/>
+            </surface> -->
+        </collision>
+        <xacro:inertial_box mass="0.001" x="${fork_base_width}" y="${fork_base_length}" z="${fork_base_height}" >
+            <origin xyz="0 0 ${(fork_base_height / 2)}" rpy="0 0 0"/>
         </xacro:inertial_box>
     </link>
@@ -370,6 +374,6 @@
             </geometry>
         </collision>
-        <xacro:inertial_box mass="${front_wheel_mass}" x="0" y="0" z="0" > <!-- TODO: set weight etc. -->
-            <origin xyz="0 0 0" rpy="0 0 0"/>
+        <xacro:inertial_box mass="0.001" x="${fork_width}" y="${fork_length}" z="${fork_height}" >
+            <origin xyz="0 0 ${(fork_height / 2)}" rpy="0 0 0"/>
         </xacro:inertial_box>
     </link>
@@ -396,6 +400,6 @@
             </geometry>
         </collision>
-        <xacro:inertial_box mass="${front_wheel_mass}" x="0" y="0" z="0" > <!-- TODO: set weight etc. -->
-            <origin xyz="0 0 0" rpy="0 0 0"/>
+        <xacro:inertial_box mass="0.001" x="${fork_width}" y="${fork_length}" z="${fork_height}" >
+            <origin xyz="0 0 ${(fork_height / 2)}" rpy="0 0 0"/>
         </xacro:inertial_box>
     </link>
@@ -407,4 +411,5 @@
     <!-- Setup ROS_CONTROL and transmission tags for the forklift robot-->
     <xacro:include filename="ros2_control.xacro"/>
+    <!-- <xacro:include filename="gazebo.xacro"/> -->
     <!-- Setup Collision Detection Plugin for the forklift robot -->
     <xacro:include filename="ros_gazebo_collision_detection_plugin.xacro"/>

File: src/forklift_robot/urdf/gazebo.xacro (robot description, xacro)
@@ -117,4 +117,5 @@
     <xacro:property name="front_wheel_radius" value="0.30" />
     <xacro:property name="front_wheel_thickness" value="0.23" /> Made up number TODO: tune this parameter -->
+     <!-- to test run: $ros2 run teleop_twist_keyboard teleop_twist_keyboard  -->
     <gazebo>
         <plugin name="diff_drive" filename="libgazebo_ros_diff_drive.so">
@@ -129,5 +130,6 @@
             <!-- Output -->
             <odometry_frame>odom</odometry_frame>
-            <robot_base_frame>base_link</robot_base_frame>
+            <!-- <robot_base_frame>base_link</robot_base_frame> -->
+            <robot_base_frame>chassis_bottom_link</robot_base_frame>
             <publish_odom>true</publish_odom>
             <publish_odom_tf>true</publish_odom_tf>
