Commit message: forklift urdf changed substantially. manual control no longer uses ros2 control's diff_drive but gazebo_diff_drive. gui_controller has Q btn to stop robot.

File: src/forklift_robot/urdf/forklift.urdf.xacro (robot description, xacro)
@@ -8,13 +8,10 @@
     <xacro:property name="chassis_top_length" value="1.59" />
     <xacro:property name="chassis_top_height" value="1.808" />
-    <!-- <xacro:property name="back_wheel_radius" value="0.221" />
-    <xacro:property name="back_wheel_thickness" value="0.221" />  -->
-    <xacro:property name="back_wheel_radius" value="0.30" />
-    <xacro:property name="back_wheel_thickness" value="0.23" /> <!-- Made up number TODO: tune this parameter -->
-    <xacro:property name="back_wheel_mass" value="0.01" /> <!-- Made up number TODO: tune this parameter -->
+    <xacro:property name="back_wheel_radius" value="0.05" />
+    <xacro:property name="back_wheel_mass" value="0.1" />
     <xacro:property name="back_wheel_length_offset" value="${(chassis_bottom_length / 2)  * (2/3)}" />
-    <xacro:property name="front_wheel_radius" value="0.30" />
-    <xacro:property name="front_wheel_thickness" value="0.23" /> <!-- Made up number TODO: tune this parameter -->
-    <xacro:property name="front_wheel_mass" value="0.005" /> <!-- Made up number TODO: tune this parameter -->
+    <xacro:property name="front_wheel_radius" value="0.05" />
+    <xacro:property name="front_wheel_thickness" value="0.04" />
+    <xacro:property name="front_wheel_mass" value="0.1" />
     <xacro:property name="front_wheel_length_offset" value="${(chassis_bottom_length / 2)}" />
     <xacro:property name="lift_body_connector_length" value="0.15" />
@@ -41,23 +38,25 @@
     <xacro:property name="camera_image_clip_near" value="0.05" /> <!-- how close the camera can see -->
     <xacro:property name="camera_image_clip_far" value="8" /> <!-- how far the camera can see -->
-    <xacro:property name="collision_detection_plugin_update_rate" value="30.0" /> <!-- how far the camera can see -->
+    <xacro:property name="collision_detection_plugin_update_rate" value="30.0" />
     <xacro:include filename="inertial_macros.xacro"/>
     <xacro:include filename="gazebo_colors.xacro"/>
     <!-- <xacro:include filename="lidar.xacro"/> -->
     <!-- <xacro:include filename="camera.xacro"/> --> <!-- Uncomment this line, and comment the line below to switch between Depth Camera and a Regular Camera -->
-    <xacro:include filename="depth_camera.xacro"/>
-    <!-- BASE LINK -->
-    <!-- <link name="base_link">
-    </link>
+    <!-- <xacro:include filename="depth_camera.xacro"/> -->
+        <!-- BASE LINK -->
+    <link name="base_link">
+        <origin xyz="0 0 0" rpy="0 0 0"/>
+    </link>
+    <!-- CHASSIS LINK -->
     <joint name="chassis_joint" type="fixed">
         <parent link="base_link"/>
         <child link="chassis_bottom_link"/>
-        <origin xyz="0 0 0"/>
-    </joint> -->
+        <origin xyz="-0.1 0 0"/>
+    </joint>
     <link name="chassis_bottom_link">
         <visual>
             <origin xyz="0 0 ${chassis_bottom_height / 2}" rpy="0 0 0"/>
             <geometry>
-                <box size="${chassis_bottom_width} ${chassis_bottom_length} ${chassis_bottom_height}" />
+                <box size="${chassis_bottom_length} ${chassis_bottom_width} ${chassis_bottom_height}" />
             </geometry>
             <material name="green">
@@ -68,32 +67,14 @@
             <origin xyz="0 0 ${chassis_bottom_height / 2}" rpy="0 0 0"/>
             <geometry>
-                <box size="${chassis_bottom_width} ${chassis_bottom_length} ${chassis_bottom_height}" />
-            </geometry>
-        </collision>
-        <xacro:inertial_box mass="1" x="${chassis_bottom_width}" y="${chassis_bottom_length}" z="${chassis_bottom_height}">
+                <box size="${chassis_bottom_length} ${chassis_bottom_width} ${chassis_bottom_height}" />
+            </geometry>
+        </collision>
+        <xacro:inertial_box mass="30" x="${chassis_bottom_length}" y="${chassis_bottom_width}" z="${chassis_bottom_height}">
             <origin xyz="0 0 ${chassis_bottom_height / 2}" rpy="0 0 0"/>
         </xacro:inertial_box>
     </link>
-    <!-- top of the chassis -->
-    <link name="chassis_top_link">
-        <visual>
-            <origin xyz="0 0 ${chassis_top_height / 2}" rpy="0 0 0"/>
-            <geometry>
-                <box size="${chassis_top_width} ${chassis_top_length} ${chassis_top_height}" />
-            </geometry>
-            <material name="red">
-                <color rgba="1 0 0 1"/>
-            </material>
-        </visual>
-        <collision>
-            <origin xyz="0 0 ${chassis_top_height / 2}" rpy="0 0 0"/>
-            <geometry>
-                <box size="${chassis_top_width} ${chassis_top_length} ${chassis_top_height}" />
-            </geometry>
-        </collision>
-        <xacro:inertial_box mass="5" x="${chassis_top_width}" y="${chassis_top_length}" z="${chassis_top_height}">
-            <origin xyz="0 0 ${chassis_top_height / 2}" rpy="0 0 0"/>
-        </xacro:inertial_box>
-    </link>
+    <gazebo reference="chassis_bottom_link">
+        <material>Gazebo/White</material>
+    </gazebo>
     <joint name="chassis_top_joint" type="fixed">
         <origin xyz="0 0 ${chassis_bottom_height}" rpy="0 0 0"/>
@@ -101,37 +82,90 @@
         <child link="chassis_top_link"/>
     </joint>
-    <!-- right_back_wheel -->
-    <!-- <link name="right_back_wheel_link">
-        <visual>
-            <geometry>
-                <cylinder radius="${back_wheel_radius}" length="${back_wheel_thickness}"/>
-            </geometry>
-            <material name="blue">
-                <color rgba="0 0 1 1"/>
-            </material>
-        </visual>
-        <collision>
-            <geometry>
-                <cylinder radius="${back_wheel_radius}" length="${back_wheel_thickness}"/>
-            </geometry>
-        </collision>
-        <xacro:inertial_cylinder mass="${back_wheel_mass}" length="${back_wheel_thickness}" radius="${back_wheel_radius}">
+    <link name="chassis_top_link">
+        <visual>
+            <origin xyz="0 0 ${chassis_top_height / 2}" rpy="0 0 0"/>
+            <geometry>
+                <box size="${chassis_top_length} ${chassis_top_width} ${chassis_top_height}" />
+            </geometry>
+            <material name="red">
+                <color rgba="1 0 0 1"/>
+            </material>
+        </visual>
+        <collision>
+            <origin xyz="0 0 ${chassis_top_height / 2}" rpy="0 0 0"/>
+            <geometry>
+                <box size="${chassis_top_length} ${chassis_top_width} ${chassis_top_height}" />
+            </geometry>
+        </collision>
+        <xacro:inertial_box mass="5" x="${chassis_top_length}" y="${chassis_top_width}" z="${chassis_top_height}">
+            <origin xyz="0 0 ${chassis_top_height / 2}" rpy="0 0 0"/>
+        </xacro:inertial_box>
+    </link>
+    <!-- LEFT WHEEL LINK -->
+    <joint name="left_wheel_joint" type="continuous">
+        <parent link="base_link"/>
+        <child link="left_wheel"/>
+        <!-- <origin xyz="0 0.175 0" rpy="-${pi/2} 0 0" /> -->
+        <origin xyz="${front_wheel_length_offset} ${(chassis_bottom_width / 2)} 0" rpy="-${pi/2} 0 0" />
+        <axis xyz="0 0 1"/>
+    </joint>
+    <link name="left_wheel">
+        <visual>
+            <geometry>
+                <cylinder radius="${front_wheel_radius}" length="${front_wheel_thickness}"/>
+            </geometry>
+            <material name="blue"/>
+        </visual>
+        <collision>
+            <geometry>
+                <cylinder radius="${front_wheel_radius}" length="${front_wheel_thickness}"/>
+            </geometry>
+        </collision>
+        <xacro:inertial_cylinder mass="${front_wheel_mass}" length="${front_wheel_thickness}" radius="${front_wheel_radius}">
             <origin xyz="0 0 0" rpy="0 0 0"/>
         </xacro:inertial_cylinder>
     </link>
-    <joint name="right_back_wheel_joint" type="continuous">
+    <gazebo reference="left_wheel">
+        <material>Gazebo/Blue</material>
+    </gazebo>
+    <!-- RIGHT FRONT WHEEL LINK -->
+    <joint name="right_wheel_joint" type="continuous">
+        <parent link="base_link"/>
+        <child link="right_wheel"/>
+        <!-- <origin xyz="0 -0.175 0" rpy="${pi/2} 0 0" /> -->
+        <origin xyz="${front_wheel_length_offset} -${(chassis_bottom_width / 2)} 0" rpy="${pi/2} 0 0" />
+        <axis xyz="0 0 -1"/>
+    </joint>
+    <link name="right_wheel">
+        <visual>
+            <geometry>
+                <cylinder radius="${front_wheel_radius}" length="${front_wheel_thickness}"/>
+            </geometry>
+            <material name="blue"/>
+        </visual>
+        <collision>
+            <geometry>
+                <cylinder radius="${front_wheel_radius}" length="${front_wheel_thickness}"/>
+            </geometry>
+        </collision>
+        <xacro:inertial_cylinder mass="${front_wheel_mass}" length="${front_wheel_thickness}" radius="${front_wheel_radius}">
+            <origin xyz="0 0 0" rpy="0 0 0"/>
+        </xacro:inertial_cylinder>
+    </link>
+    <gazebo reference="right_wheel">
+        <material>Gazebo/Blue</material>
+    </gazebo>
+    <!-- CASTER WHEEL LINK -->
+    <joint name="caster_wheel_joint" type="fixed">
         <parent link="chassis_bottom_link"/>
-        <child link="right_back_wheel_link"/>
-        <origin xyz="${(chassis_bottom_width / 2) - (back_wheel_thickness / 2)} -${back_wheel_length_offset} 0" rpy="0 -${pi/2} 0" />
-        <axis xyz="0 0 1"/>
-    </joint> -->
-    <link name="back_wheel_link">
+        <child link="caster_wheel"/>
+        <origin xyz="-${back_wheel_length_offset} 0 0" />
+    </joint>
+    <link name="caster_wheel">
         <visual>
             <geometry>
                 <sphere radius="${back_wheel_radius}"/>
             </geometry>
-            <material name="blue">
-                <color rgba="0 0 1 1"/>
-            </material>
+            <material name="black"/>
         </visual>
         <collision>
@@ -144,115 +178,26 @@
         </xacro:inertial_sphere>
     </link>
-    <!-- <joint name="back_wheel_joint" type="fixed">
-        <parent link="chassis_bottom_link"/>
-        <child link="back_wheel_link"/>
-        <origin xyz=" 0 -${back_wheel_length_offset} 0" rpy="0 -${pi/2} 0" />
-    </joint> -->
-    <joint name="back_wheel_joint" type="fixed">
-        <parent link="chassis_bottom_link"/>
-        <child link="back_wheel_link"/>
-        <origin xyz=" 0 -${back_wheel_length_offset} 0" />
-    </joint>
-    <!-- Wheel Frictions -->
-    <gazebo reference="back_wheel_link">
-        <material>Gazebo/White</material>
+    <!-- FRICTION VALUES -->
+    <gazebo reference="caster_wheel">
+        <material>Gazebo/Black</material>
         <mu1 value="0.001"/>
         <mu2 value="0.001"/>
     </gazebo>
-    <gazebo reference="right_front_wheel_link">
-        <material>Gazebo/White</material>
-        <mu1 value="1.0"/>
-        <mu2 value="0.25"/>
-    </gazebo>
-    <gazebo reference="left_front_wheel_link">
-        <material>Gazebo/White</material>
-        <mu1 value="1.0"/>
-        <mu2 value="0.25"/>
-    </gazebo>
-    <!-- left_back_wheel -->
-    <!-- <link name="left_back_wheel_link">
-        <visual>
-            <geometry>
-                <cylinder radius="${back_wheel_radius}" length="${back_wheel_thickness}"/>
-            </geometry>
-            <material name="blue">
-                <color rgba="0 0 1 1"/>
-            </material>
-        </visual>
-        <collision>
-            <geometry>
-                <cylinder radius="${back_wheel_radius}" length="${back_wheel_thickness}"/>
-            </geometry>
-        </collision>
-        <xacro:inertial_cylinder mass="${back_wheel_mass}" length="${back_wheel_thickness}" radius="${back_wheel_radius}">
-            <origin xyz="0 0 0" rpy="0 0 0"/>
-        </xacro:inertial_cylinder>
-    </link>
-    <joint name="left_back_wheel_joint" type="continuous">
-        <parent link="chassis_bottom_link"/>
-        <child link="left_back_wheel_link"/>
-        <origin xyz="${- (chassis_bottom_width / 2) + (back_wheel_thickness / 2)} -${back_wheel_length_offset} 0" rpy="0 -${pi/2} 0" />
-        <axis xyz="0 0 1"/>
-    </joint> -->
-    <!-- right_front_wheel -->
-    <link name="right_front_wheel_link">
-        <visual>
-            <geometry>
-                <cylinder radius="${front_wheel_radius}" length="${front_wheel_thickness}"/>
-            </geometry>
-            <material name="blue">
-                <color rgba="0 0 1 1"/>
-            </material>
-        </visual>
-        <collision>
-            <geometry>
-                <cylinder radius="${front_wheel_radius}" length="${front_wheel_thickness}"/>
-            </geometry>
-        </collision>
-        <xacro:inertial_cylinder mass="${front_wheel_mass}" length="${front_wheel_thickness}" radius="${front_wheel_radius}">
-            <origin xyz="0 0 0" rpy="0 0 0"/>
-        </xacro:inertial_cylinder>
-    </link>
-    <joint name="right_front_wheel_joint" type="continuous">
-        <parent link="chassis_bottom_link"/>
-        <child link="right_front_wheel_link"/>
-        <!-- <origin xyz="${(chassis_bottom_width / 2) - (front_wheel_thickness / 2)} ${front_wheel_length_offset} 0" rpy="0 ${pi/2} 0" /> -->
-        <origin xyz="${(chassis_bottom_width / 2)} ${front_wheel_length_offset} 0" rpy="0 ${pi/2} 0" />
-        <axis xyz="0 0 -1"/>
-        <dynamics damping="0.2"/>
-    </joint>
-    <!-- left_front_wheel -->
-    <link name="left_front_wheel_link">
-        <visual>
-            <geometry>
-                <cylinder radius="${front_wheel_radius}" length="${front_wheel_thickness}"/>
-            </geometry>
-            <material name="blue">
-                <color rgba="0 0 1 1"/>
-            </material>
-        </visual>
-        <collision>
-            <geometry>
-                <cylinder radius="${front_wheel_radius}" length="${front_wheel_thickness}"/>
-            </geometry>
-        </collision>
-        <xacro:inertial_cylinder mass="${front_wheel_mass}" length="${front_wheel_thickness}" radius="${front_wheel_radius}">
-            <origin xyz="0 0 0" rpy="0 0 0"/>
-        </xacro:inertial_cylinder>
-    </link>
-    <joint name="left_front_wheel_joint" type="continuous">
-        <parent link="chassis_bottom_link"/>
-        <child link="left_front_wheel_link"/>
-        <!-- <origin xyz="${ -(chassis_bottom_width / 2) + (front_wheel_thickness / 2)} ${front_wheel_length_offset} 0" rpy="0 -${pi/2} 0" /> -->
-        <origin xyz="${ -(chassis_bottom_width / 2)} ${front_wheel_length_offset} 0" rpy="0 -${pi/2} 0" />
-        <axis xyz="0 0 1"/>
-        <dynamics damping="0.2"/>
-    </joint>
-    <!-- lift_base -->
+    <gazebo reference="right_wheel">
+        <material>Gazebo/Black</material>
+        <mu1 value="10.0"/>
+        <mu2 value="10.0"/>
+    </gazebo>
+    <gazebo reference="left_wheel">
+        <material>Gazebo/Black</material>
+        <mu1 value="10.0"/>
+        <mu2 value="10.0"/>
+    </gazebo>
+     <!-- LIFT BASE LINK-->
     <link name="lift_base_link">
         <visual>
             <origin xyz="0 0 ${lift_base_height / 2}" rpy="0 0 0"/>
             <geometry>
-                <box size="${chassis_bottom_width} ${lift_base_length} ${lift_base_height}"/>
+                <box size="${lift_base_length} ${chassis_bottom_width} ${lift_base_height}"/>
             </geometry>
             <material name="red">
@@ -263,5 +208,5 @@
             <origin xyz="0 0 ${lift_base_height / 2}" rpy="0 0 0"/>
             <geometry>
-                <box size="${chassis_bottom_width} ${lift_base_length} ${lift_base_height}"/>
+                <box size="${lift_base_length} ${chassis_bottom_width} ${lift_base_height}"/>
             </geometry>
             <!-- Added by me (surface tag) to prevent fork falling down issue -->
@@ -280,5 +225,5 @@
             </surface> -->
         </collision>
-        <xacro:inertial_box mass="${0.001}" x="${chassis_bottom_width}" y="${lift_base_length}" z="${lift_base_height}" >
+        <xacro:inertial_box mass="${0.001}" x="${lift_base_length}" y="${chassis_bottom_width}" z="${lift_base_height}" >
             <origin xyz="0 0 ${lift_base_height / 2}" rpy="0 0 0"/>
         </xacro:inertial_box>
@@ -287,12 +232,12 @@
         <parent link="chassis_bottom_link"/>
         <child link="lift_base_link"/>
-        <origin xyz="0 ${(chassis_bottom_length / 2) + lift_body_connector_length + (lift_base_length / 2)} 0" rpy="0 0 0" />
-    </joint>
-    <!-- lift_body_connector -->
+        <origin xyz="${(chassis_bottom_length / 2) + lift_body_connector_length + (lift_base_length / 2)} 0 0" rpy="0 0 0" />
+    </joint>
+    <!-- LIFT BODY CONNECTOR LINK -->
     <link name="lift_body_connector_link">
         <visual>
             <origin xyz="0 0 ${(lift_body_connector_height / 2)}" rpy="0 0 0"/>
             <geometry>
-                <box size="${chassis_bottom_width} ${lift_body_connector_length} ${lift_body_connector_height}"/>
+                <box size="${lift_body_connector_length} ${chassis_bottom_width} ${lift_body_connector_height}"/>
             </geometry>
             <material name="blue">
@@ -303,8 +248,8 @@
             <origin xyz="0 0 ${(lift_body_connector_height / 2)}" rpy="0 0 0"/>
             <geometry>
-                <box size="${chassis_bottom_width} ${lift_body_connector_length} ${lift_body_connector_height}"/>
-            </geometry>
-        </collision>
-        <xacro:inertial_box mass="${0.001}" x="${chassis_bottom_width}" y="${lift_body_connector_length}" z="${lift_body_connector_height}" >
+                <box size="${lift_body_connector_length} ${chassis_bottom_width} ${lift_body_connector_height}"/>
+            </geometry>
+        </collision>
+        <xacro:inertial_box mass="${0.001}" x="${lift_body_connector_length}" y="${chassis_bottom_width}" z="${lift_body_connector_height}" >
             <origin xyz="0 0 ${(lift_body_connector_height / 2)}" rpy="0 0 0"/>
         </xacro:inertial_box>
@@ -313,12 +258,12 @@
         <parent link="chassis_bottom_link"/>
         <child link="lift_body_connector_link"/>
-        <origin xyz="0 ${(chassis_bottom_length / 2) + (lift_body_connector_length / 2)} 0" rpy="0 0 0" />
-    </joint>
-    <!-- fork_base -->
+        <origin xyz="${(chassis_bottom_length / 2) + (lift_body_connector_length / 2)} 0 0" rpy="0 0 0" />
+    </joint>
+    <!-- FORK BASE LINK -->
     <link name="fork_base_link">
         <visual>
             <origin xyz="0 0 ${(fork_base_height / 2)}" rpy="0 0 0"/>
             <geometry>
-                <box size="${fork_base_width} ${fork_base_length} ${fork_base_height}"/>
+                <box size="${fork_base_length} ${fork_base_width} ${fork_base_height}"/>
             </geometry>
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
File: src/forklift_robot/urdf/gazebo.xacro (robot description, xacro)
@@ -118,10 +118,12 @@
     <xacro:property name="front_wheel_thickness" value="0.23" /> Made up number TODO: tune this parameter -->
      <!-- to test run: $ros2 run teleop_twist_keyboard teleop_twist_keyboard  -->
+    <!-- Refer to https://classic.gazebosim.org/tutorials?tut=ros_gzplugins for diff_drive's parameters -->
     <gazebo>
         <plugin name="diff_drive" filename="libgazebo_ros_diff_drive.so">
             <!-- Wheel Information -->
-            <left_joint>left_front_wheel_joint</left_joint>
-            <right_joint>right_front_wheel_joint</right_joint>
-            <wheel_separation>${chassis_bottom_width - (2*front_wheel_thickness)}</wheel_separation>
+            <left_joint>left_wheel_joint</left_joint>
+            <right_joint>right_wheel_joint</right_joint>
+            <wheel_separation>${chassis_bottom_width}</wheel_separation>
+            <!-- <wheel_separation>0.35</wheel_separation> -->
             <wheel_diameter>${front_wheel_radius * 2}</wheel_diameter>
             <!-- Limits -->
@@ -130,6 +132,5 @@
             <!-- Output -->
             <odometry_frame>odom</odometry_frame>
-            <!-- <robot_base_frame>base_link</robot_base_frame> -->
-            <robot_base_frame>chassis_bottom_link</robot_base_frame>
+            <robot_base_frame>base_link</robot_base_frame>
             <publish_odom>true</publish_odom>
             <publish_odom_tf>true</publish_odom_tf>
