Commit message: depth_camera_raw_image_subscriber refactored

File: src/forklift_robot/urdf/depth_camera.xacro (robot description, xacro)
@@ -16,5 +16,5 @@
         <parent link="fork_base_link"/>
         <child link="camera_link"/>
-        <origin xyz="${fork_base_length / 2} ${fork_base_length / 2} ${fork_base_length / 2}" rpy="0 0 ${pi / 2}"/> <!-- TODO: when the front of the robot faces x-axis(instead of current y-axis) change to rpy="0 0 0"-->
+        <origin xyz="${fork_base_length / 2} ${fork_base_length / 2} ${fork_base_length / 2}" rpy="0 0 0"/>
     </joint>
     <!-- Convert ros coordinate system to generally used image coordinate system -->

File: src/forklift_robot/urdf/forklift.urdf.xacro (robot description, xacro)
@@ -43,5 +43,5 @@
     <!-- <xacro:include filename="lidar.xacro"/> -->
     <!-- <xacro:include filename="camera.xacro"/> --> <!-- Uncomment this line, and comment the line below to switch between Depth Camera and a Regular Camera -->
-    <!-- <xacro:include filename="depth_camera.xacro"/> -->
+    <xacro:include filename="depth_camera.xacro"/>
         <!-- BASE LINK -->
     <link name="base_link">
